File: ACS Fullscale.kicad_sch (KiCad schematic)
At the start: 18 parts, among them J1 Pulse-20, J2 Conn_01x02, U1 SN65HVD230, U11 R-78E5.0-1.0, U2 MS5611-01BA, U4 Teensy4.1, U5 TPS62202DBV, U6 BHI360, U7 TXS0108EPW

Commit message: hi
Parts:
- added U3: 4001, symbol 4xxx_IEEE:4001
Changed lines of the file:
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@@
+	)
+	(symbol
+		(lib_id "4xxx_IEEE:4001")
+		(at 81.28 144.78 0)
+		(unit 1)
+		(exclude_from_sim no)
+		(in_bom yes)
+		(on_board yes)
+		(dnp no)
+		(fields_autoplaced yes)
+		(property "Reference" "U3"
+			(at 90.17 138.3598 0)
+			(effects
+				(font
+					(size 1.27 1.27)
+				)
+			)
+		)
+		(property "Value" "4001"
+			(at 90.17 140.8998 0)
+			(effects
+				(font
+					(size 1.27 1.27)
+				)
+			)
+		)
+		(property "Footprint" ""
+			(at 81.28 144.78 0)
+			(effects
+				(font
+					(size 1.27 1.27)
+				)
+				(hide yes)
+			)
+		)
+		(property "Datasheet" ""
+			(at 81.28 144.78 0)
+			(effects
+				(font
+					(size 1.27 1.27)
+				)
+				(hide yes)
+			)
+		)
+		(property "Description" ""
+			(at 81.28 144.78 0)
+			(effects
+				(font
+					(size 1.27 1.27)
+				)
+				(hide yes)
+			)
+		)
+		(pin "9"
+		)
+		(pin "12"
+		)
+		(pin "10"
+		)
+		(pin "13"
+		)
+		(pin "11"
+		)
+		(pin "8"
+		)
+		(pin "4"
+		)
+		(pin "6"
+		)
+		(pin "5"
+		)
+		(pin "3"
+		)
+		(pin "2"
+		)
+		(pin "1"
+		)
+		(pin "7"
+		)
+		(pin "14"
+		)
+		(instances
+			(project ""
+				(path "/51f244b9-9601-4f29-b08e-b866e02fd2b7"
+					(reference "U3")
+					(unit 1)
+				)
+			)
+		)
 	)
 	(symbol
