File: CM5_HighSpeed.kicad_sch (KiCad schematic)
At the start: 19 parts, among them J10 Conn_01x22_Female, J11 THD-02-R, J12 USB3_A, J13 690-019-298-412, J14 690-019-298-412, J9 Conn_01x22_Female, U15 AP22653W6, U16 RT9742SNGV

Commit message: A lot of stuff
Parts:
- removed C22, C24, C25: 10u, Capacitor_SMD:C_0805_2012Metric, symbol Device:C
- removed C23: 100uF, Capacitor_Tantalum_SMD:CP_EIA-7343-31_Kemet-D, symbol Device:C_Polarized
- removed C26, C27: 100n, Capacitor_SMD:C_0402_1005Metric, symbol Device:C
- removed J10, J9: Conn_01x22_Female, CM5IO:Hirose_FH12-22S-0.5SH_1x22-1MP_P0.50mm_Horizontal, symbol Connector:Conn_01x22_Socket
- removed J11: THD-02-R, Connector_PinHeader_2.54mm:PinHeader_2x02_P2.54mm_Vertical, symbol Connector_Generic:Conn_02x02_Odd_Even
- removed J12: USB3_A, CM5IO:MTCONN_UBAF30-D2011, symbol CM5IO:USB3_A
- removed J13, J14: 690-019-298-412, CM5IO:EDAC 690-019-298-412, symbol CM5IO:HDMI_A_1.4
- removed R13: 15K 1%, Resistor_SMD:R_0402_1005Metric, symbol Device:R
- removed R14, R15, R16: 2.2K 1%, Resistor_SMD:R_0402_1005Metric, symbol Device:R
- removed U15: AP22653W6, Package_TO_SOT_SMD:SOT-23-6, symbol CM5IO:AP2553W6
- removed U16: RT9742SNGV, Package_TO_SOT_SMD:TSOT-23_HandSoldering, symbol CM5IO:RT9742SNGV
Connections:
- no-connect marks 4 -> 0
Other:
- note removed: "Current Limit switch"
- note removed: "DSI/CSI Connectors"
- note removed: "Jumpers to be fitted if DPHY1 is used"
- note removed: "Stacked USB connectors"
- note removed: "USB 3 Pairs P/N swapped to help routing"
