File: CM5_GPIO.kicad_sch (KiCad schematic)
At the start: 29 parts, among them J3 Conn_02x07_Odd_Even, J4 Conn_01x03, J5 JST_SHBM04B-SRSS-TB, J6 THD-20-R, J7 THD-02-R, J8 Micro_SD_Card_Det, SW1 Right angle Tact button, U12 TPD4EUSB30, U13 RT9742GGJ5, U14 MagJack-A70-112-331N126, U3 TPD4EUSB30

Commit message: A lot of stuff
Parts:
- removed BT1: Battery_Cell, CM5IO:BatteryHolder_Keystone_3034_1x20mm, symbol Device:Battery_Cell
- removed J4: Conn_01x03, Connector_PinHeader_2.54mm:PinHeader_1x03_P2.54mm_Vertical, symbol Connector_Generic:Conn_01x03
- removed J5: JST_SHBM04B-SRSS-TB, Connector_JST:JST_SH_BM04B-SRSS-TB_1x04-1MP_P1.00mm_Vertical, symbol Connector_Generic:Conn_01x04
- removed J6: THD-20-R, Connector_PinHeader_2.54mm:PinHeader_2x20_P2.54mm_Vertical, symbol Connector_Generic:Conn_02x20_Odd_Even
- removed R2: 10K 1%, Resistor_SMD:R_0402_1005Metric, symbol Device:R
- removed R3: 0R, Resistor_SMD:R_0805_2012Metric_Pad1.20x1.40mm_HandSolder, symbol Device:R
- removed R8: nf, Resistor_SMD:R_0805_2012Metric_Pad1.20x1.40mm_HandSolder, symbol Device:R
- removed SW1: Right angle Tact button, Button_Switch_THT:SW_Tactile_SPST_Angled_PTS645Vx58-2LFS, symbol Switch:SW_Push
- removed TP1, TP2, TP3, TP4: TestPoint, TestPoint:TestPoint_Pad_2.0x2.0mm, symbol Connector:TestPoint
Connections:
- net GPIO_VREF is gone; now on net +3V3: Module1.78 (GPIO_VREF(1.8v/3.3v_Input))
- net GND: now also Module1.92 (PWR_BUT)
- net PWR_BUT: no longer Module1.92 (PWR_BUT)
- net +3.3v renamed +3V3
- net GPIO14 renamed TX
- net GPIO15 renamed RX
Other:
- note removed: "40Way GPIO Header"
- note removed: "FAN connector"
- note removed: "GPIO Voltage select"
- note removed: "Not Fitted header"
- note removed: "R2 : Pullup added for Fans that don't have a strong internal pullup"

Commit message: ryan
Parts:
- added J6: Conn_01x05, Connector_PinHeader_2.54mm:PinHeader_1x05_P2.54mm_Vertical, symbol Connector_Generic:Conn_01x05
- added J9: Conn_01x02, Connector_PinHeader_2.54mm:PinHeader_1x02_P2.54mm_Vertical, symbol Connector_Generic:Conn_01x02
Connections:
- net GPIO10: now also J6.1 (Pin_1)
- net GPIO11: now also J6.3 (Pin_3)
- net GPIO2: now also J9.1 (Pin_1)
- net GPIO3: now also J9.2 (Pin_2)
- net GPIO7: now also J6.4 (Pin_4)
- net GPIO8: now also J6.5 (Pin_5)
- net GPIO9: now also J6.2 (Pin_2)
