File: BNO086.kicad_sch (KiCad schematic)
At the start: 14 parts, among them U10 BNO086, U9 BME280, Y1 32.768k

Commit message: fix lib
Parts:
- removed U10: BNO086, Package_LGA:LGA-28_5.2x3.8mm_P0.5mm, symbol Sensor_Motion:BNO086
- added U10: BNO086, Package_LGA:LGA-28_5.2x3.8mm_P0.5mm, symbol ACS_symbol_Library:BNO086
Connections:
- net +3V3: now also U10.28 (VDDIO), U10.3 (VDD), U10.5 (PS1)
- net BT: now also U10.4 (~{BOOT_LOAD_PIN})
- net CS: now also U10.18 (H_CSN)
- net GND: now also U10.10 (CLKSEL0), U10.2 (GND), U10.25 (GNDIO)
- net INT: now also U10.14 (INT)
- net MISO: now also U10.20 (H_SDA/H_MISO/TX)
- net MOSI: now also U10.17 (SA0/H_MOSI)
- net RST: now also U10.11 (~{RESET})
- net SCK: now also U10.19 (H_SCL/SCK/RX)
- net SCL: now also U10.15 (ENV_SCL)
- net SDA: now also U10.16 (ENV_SDA)
- net WAKE: now also U10.6 (PS0)
- net at C18.1, Y1.2: now also U10.26 (XOUT32)
- net at C17.1, Y1.1: now also U10.27 (XIN32)
- net at C16.1: now also U10.9 (CAP)
Changed lines of the file:
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@@
+	)
+	(symbol
+		(lib_id "ACS_symbol_Library:BNO086")
+		(at 193.04 99.06 0)
+		(unit 1)
+		(exclude_from_sim no)
+		(in_bom yes)
+		(on_board yes)
+		(dnp no)
+		(fields_autoplaced yes)
+		(property "Reference" "U10"
+			(at 197.7233 73.66 0)
+			(effects
+				(font
+					(size 1.27 1.27)
+				)
+				(justify left)
+			)
+		)
+		(property "Value" "BNO086"
+			(at 197.7233 76.2 0)
+			(effects
+				(font
+					(size 1.27 1.27)
+				)
+				(justify left)
+			)
+		)
+		(property "Footprint" "Package_LGA:LGA-28_5.2x3.8mm_P0.5mm"
+			(at 199.39 106.68 0)
+			(effects
+				(font
+					(size 1.27 1.27)
+				)
+				(justify left)
+				(hide yes)
+			)
+		)
+		(property "Datasheet" "https://mm.digikey.com/Volume0/opasdata/d220001/medias/docus/6531/BNO080_085_Datasheet-3196201.pdf"
+			(at 193.04 93.98 0)
+			(effects
+				(font
+					(size 1.27 1.27)
+				)
+				(hide yes)
+			)
+		)
+		(property "Description" "Intelligent 9-axis absolute orientation sensor, LGA-28"
+			(at 193.04 93.98 0)
+			(effects
+				(font
+					(size 1.27 1.27)
+				)
+				(hide yes)
+			)
+		)
+		(pin "9"
+		)
+		(pin "24"
+		)
+		(pin "6"
+		)
+		(pin "23"
+		)
+		(pin "5"
+		)
+		(pin "1"
+		)
+		(pin "14"
+		)
+		(pin "7"
+		)
+		(pin "4"
+		)
+		(pin "10"
+		)
+		(pin "8"
+		)
+		(pin "20"
+		)
+		(pin "19"
+		)
+		(pin "18"
+		)
+		(pin "17"
+		)
+		(pin "15"
+		)
+		(pin "16"
+		)
+		(pin "3"
+		)
+		(pin "2"
+		)
+		(pin "28"
+		)
+		(pin "25"
+		)
+		(pin "26"
+		)
+		(pin "27"
+		)
+		(pin "22"
+		)
+		(pin "13"
+		)
+		(pin "11"
+		)
+		(pin "12"
+		)
+		(pin "21"
+		)
+		(instances
+			(project ""
+				(path "/51f244b9-9601-4f29-b08e-b866e02fd2b7/d0a5d860-5b4f-45de-b012-9a4b91f44335"
+					(reference "U10")
+					(unit 1)
+				)
+			)
+		)
 	)
 	(symbol
@@
 					(unit 1)
 				)
-			)
-		)
-	)
-	(symbol
-		(lib_id "Sensor_Motion:BNO086")
-		(at 193.04 99.06 0)
-		(unit 1)
-		(exclude_from_sim no)
-		(in_bom yes)
-		(on_board yes)
-		(dnp no)
-		(fields_autoplaced yes)
-		(property "Reference" "U10"
-			(at 197.7233 73.66 0)
-			(effects
-				(font
-					(size 1.27 1.27)
-				)
-				(justify left)
-			)
-		)
-		(property "Value" "BNO086"
-			(at 197.7233 76.2 0)
-			(effects
-				(font
-					(size 1.27 1.27)
-				)
-				(justify left)
-			)
-		)
-		(property "Footprint" "Package_LGA:LGA-28_5.2x3.8mm_P0.5mm"
-			(at 199.39 106.68 0)
-			(effects
-				(font
-					(size 1.27 1.27)
-				)
-				(justify left)
-				(hide yes)
-			)
-		)
-		(property "Datasheet" "https://mm.digikey.com/Volume0/opasdata/d220001/medias/docus/6531/BNO080_085_Datasheet-3196201.pdf"
-			(at 193.04 93.98 0)
-			(effects
-				(font
-					(size 1.27 1.27)
-				)
-				(hide yes)
-			)
-		)
-		(property "Description" "Intelligent 9-axis absolute orientation sensor, LGA-28"
-			(at 193.04 93.98 0)
-			(effects
-				(font
-					(size 1.27 1.27)
-				)
-				(hide yes)
-			)
-		)
-		(pin "7"
-		)
-		(pin "8"
-		)
-		(pin "3"
-		)
-		(pin "2"
-		)
-		(pin "28"
-		)
-		(pin "25"
-		)
-		(pin "12"
-		)
-		(pin "10"
-		)
-		(pin "4"
-		)
-		(pin "20"
-		)
-		(pin "19"
-		)
-		(pin "1"
-		)
-		(pin "16"
-		)
-		(pin "15"
-		)
-		(pin "17"
-		)
-		(pin "18"
-		)
-		(pin "11"
-		)
-		(pin "14"
-		)
-		(pin "21"
-		)
-		(pin "13"
-		)
-		(pin "22"
-		)
-		(pin "23"
-		)
-		(pin "9"
-		)
-		(pin "27"
-		)
-		(pin "24"
-		)
-		(pin "26"
-		)
-		(pin "6"
-		)
-		(pin "5"
-		)
-		(instances
-			(project ""
-				(path "/51f244b9-9601-4f29-b08e-b866e02fd2b7/d0a5d860-5b4f-45de-b012-9a4b91f44335"
-					(reference "U10")
-					(unit 1)
-				)

Commit message: lots
Parts:
- removed C12, C13, C14, C15, C16: 100nF, Capacitor_SMD:C_0603_1608Metric, symbol Device:C_Small
- removed C17, C18: 22pF, Capacitor_SMD:C_0603_1608Metric, symbol Device:C_Small
- removed R4, R5: 4.7k, Resistor_SMD:R_0603_1608Metric, symbol Device:R_Small_US
- removed R6, R7: 10k, Resistor_SMD:R_0603_1608Metric, symbol Device:R_Small_US
- removed U10: BNO086, Package_LGA:LGA-28_5.2x3.8mm_P0.5mm, symbol ACS_symbol_Library:BNO086
- removed U9: BME280, Package_LGA:Bosch_LGA-8_2.5x2.5mm_P0.65mm_ClockwisePinNumbering, symbol Sensor:BME280
- removed Y1: 32.768k, Crystal:Crystal_SMD_3215-2Pin_3.2x1.5mm, symbol Device:Crystal_Small
Other:
- note removed: "Things I changed: These are all very not obvious and you have dig through the datasheet but I decreased the SDA/SCL pullup resistors to 4.7k since we are only using 1 additional integrated sensor. Also, although on the typical application schematic in the datasheet has clksel0, you actually need to connect it to ground (user selectable pin). Finally, to make the SPI work properly without a requir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"
